File: Tarea #3/Aislador/Aislador.kicad_pcb (KiCad board)
At the start: 2 copper layers, 0 parts

Commit message: Aislador
Parts:
- added C10: GRM21BR71H104KA01L, SamacSys_Parts:CAPC2012X145N, F.Cu at (166.0, 74.2)
- added C11: GRM21BR71H104KA01L, SamacSys_Parts:CAPC2012X145N, F.Cu at (166.0, 77.1)
- added C2: GRM21BR61C106KE15L, SamacSys_Parts:CAPC2012X145N, F.Cu at (162.0, 65.8)
- added C3: GRM21BR61C106KE15L, SamacSys_Parts:CAPC2012X145N, F.Cu at (162.0, 68.6)
- added C4: GRM21BR71H104KA01L, SamacSys_Parts:CAPC2012X145N, F.Cu at (162.0, 71.4)
- added C5: GRM21BR71H104KA01L, SamacSys_Parts:CAPC2012X145N, F.Cu at (162.0, 74.2)
- added C6: GRM21BR71H104KA01L, SamacSys_Parts:CAPC2012X145N, F.Cu at (162.0, 77.1)
- added C7: GRM21BR71H104KA01L, SamacSys_Parts:CAPC2012X145N, F.Cu at (166.0, 65.8)
- added C8: GRM21BR71H104KA01L, SamacSys_Parts:CAPC2012X145N, F.Cu at (166.0, 68.6)
- added C9: GRM21BR71H104KA01L, SamacSys_Parts:CAPC2012X145N, F.Cu at (166.0, 71.4)
- added D1: IR26-21C_L110_TR8, LED_SMD:LED_1206_3216Metric, F.Cu at (165.6, 83.1)
- added D2: IR26-21C_L110_TR8, LED_SMD:LED_1206_3216Metric, F.Cu at (165.6, 86.5)
- added IC1: ADUM5000ARWZ, SamacSys_Parts:SOIC127P1032X265-16N, F.Cu at (156.3, 87.5)
- added IC2: NUP2202W1T2G, SamacSys_Parts:SOT65P210X110-6N, F.Cu at (165.1, 90.1)
- added IC3: NUP2202W1T2G, SamacSys_Parts:SOT65P210X110-6N, F.Cu at (165.1, 93.8)
- added IC4: ADUM4160BRWZ, SamacSys_Parts:SOIC127P1032X265-16N, F.Cu at (156.3, 99.5)
- added J1: 87520-0010BLF, SamacSys_Parts:875200010BLF, F.Cu at (137.7, 66.9)
- added J2: USB-B-S-F-B-TH-R, SamacSys_Parts:USBBSFBTHR, F.Cu at (141.9, 84.1)
- added R10: ERJ-6GEY0R00V, SamacSys_Parts:RESC2012X70N, F.Cu at (153.2, 74.7)
- added R11: ERJ-6GEY0R00V, SamacSys_Parts:RESC2012X70N, F.Cu at (153.2, 77.6)
- added R12: ERJ-6GEY0R00V, SamacSys_Parts:RESC2012X70N, F.Cu at (157.8, 65.8)
- added R13: ERJ-6GEY0R00V, SamacSys_Parts:RESC2012X70N, F.Cu at (157.8, 68.8)
- added R14: ERJ-6GEY0R00V, SamacSys_Parts:RESC2012X70N, F.Cu at (157.8, 71.7)
- added R15: ERJ-6GEY0R00V, SamacSys_Parts:RESC2012X70N, F.Cu at (157.8, 74.7)
- added R16: ERJ-6GEY0R00V, SamacSys_Parts:RESC2012X70N, F.Cu at (157.8, 77.6)
- added R2: ERJ-6ENF1002V, SamacSys_Parts:ERJ6ENF1000V, F.Cu at (134.6, 102.9)
- added R3: ERJ-6GEY0R00V, SamacSys_Parts:RESC2012X70N, F.Cu at (153.2, 65.8)
- added R8: ERJ-6GEY0R00V, SamacSys_Parts:RESC2012X70N, F.Cu at (153.2, 68.8)
- added R9: ERJ-6GEY0R00V, SamacSys_Parts:RESC2012X70N, F.Cu at (153.2, 71.7)
