File: Tarea #3/Aislador/Aislador.kicad_sch (KiCad schematic)
At the start: 0 parts

Commit message: Libreria
Parts:
- added C1: GRM21BR71H104KA01L, SamacSys_Parts:CAPC2012X145N, symbol SamacSys_Parts:GRM21BR71H104KA01L
- added C2: GRM21BR61C106KE15L, SamacSys_Parts:CAPC2012X145N, symbol SamacSys_Parts:GRM21BR61C106KE15L
- added IC1: ADUM4160BRWZ, SamacSys_Parts:SOIC127P1032X265-16N, symbol SamacSys_Parts:ADUM4160BRWZ
- added IC2: ADUM5000ARWZ, SamacSys_Parts:SOIC127P1032X265-16N, symbol SamacSys_Parts:ADUM5000ARWZ
- added IC3: NUP2202W1T2G, SamacSys_Parts:SOT65P210X110-6N, symbol SamacSys_Parts:NUP2202W1T2G
- added J1: 87520-0010BLF, SamacSys_Parts:875200010BLF, symbol SamacSys_Parts:87520-0010BLF
- added J2: USB-B-S-F-B-TH-R, SamacSys_Parts:USBBSFBTHR, symbol SamacSys_Parts:USB-B-S-F-B-TH-R
- added R1: ERJ-6GEY0R00V, SamacSys_Parts:RESC2012X70N, symbol SamacSys_Parts:ERJ-6GEY0R00V
- added R2: ERJ-6ENF1002V, SamacSys_Parts:ERJ6ENF1000V, symbol SamacSys_Parts:ERJ-6ENF1002V

Commit message: Aislador
Parts:
- added C3, C4, C5, C6, C7, C8, C9: C_Small, symbol Device:C_Small
Connections:
- net at J2.1: now also IC1.3 (VDD1), IC1.4 (PDEN), C3.1
- net at IC1.2 (GND1_1): now also C3.2
- net at IC2.1 (VDD1_1): now also IC2.6 (RCSEL), IC2.7 (VDD1_2), C4.2, C5.2, C6.1
- net at IC2.10 (VISO_1): now also IC2.11 (NC_2), IC2.13 (VSEL), IC2.16 (VISO_2), C7.2, C8.1, C9.2
- net GND_B: now reaches IC2.15 (GNDISO_2)
- net GND_B: now also IC2.9 (GNDISO_1), C7.1, C8.2, C9.1
- net GND_A: now reaches IC2.2 (GND1_1)
- net GND_A: now also IC2.8 (GND1_2), C4.1, C5.1, C6.2
Other:
- moved on the sheet: C1, C2, IC1, IC2, IC3, J1, J2, R1, R2

Commit message: Aislador
Parts:
- removed C1: GRM21BR71H104KA01L, SamacSys_Parts:CAPC2012X145N, symbol SamacSys_Parts:GRM21BR71H104KA01L
- removed C2: GRM21BR61C106KE15L, SamacSys_Parts:CAPC2012X145N, symbol SamacSys_Parts:GRM21BR61C106KE15L
- removed C3, C4, C5, C6, C7, C8, C9: C_Small, symbol Device:C_Small
- removed IC1: ADUM4160BRWZ, SamacSys_Parts:SOIC127P1032X265-16N, symbol SamacSys_Parts:ADUM4160BRWZ
- removed IC2: ADUM5000ARWZ, SamacSys_Parts:SOIC127P1032X265-16N, symbol SamacSys_Parts:ADUM5000ARWZ
- removed IC3: NUP2202W1T2G, SamacSys_Parts:SOT65P210X110-6N, symbol SamacSys_Parts:NUP2202W1T2G
- removed J1: 87520-0010BLF, SamacSys_Parts:875200010BLF, symbol SamacSys_Parts:87520-0010BLF
- removed J2: USB-B-S-F-B-TH-R, SamacSys_Parts:USBBSFBTHR, symbol SamacSys_Parts:USB-B-S-F-B-TH-R
- removed R1: ERJ-6GEY0R00V, SamacSys_Parts:RESC2012X70N, symbol SamacSys_Parts:ERJ-6GEY0R00V
- removed R2: ERJ-6ENF1002V, SamacSys_Parts:ERJ6ENF1000V, symbol SamacSys_Parts:ERJ-6ENF1002V
- added C1, C14: 470uF/16v, Samacsys:EEE1AA220WR, symbol Samacsys:EEE-FN1C470UR
- added C10, C11, C12, C13, C15, C3: .1uF, Samacsys:CAPC1608X90N, symbol Samacsys:0603YC104J4T2A
- added C16, C2: 10uF, Samacsys:CAPC1608X102N, symbol Samacsys:0603YD106KAT2A
- added D1, D2: USBLC6-2SC6, EasyEDA:SOT-23-6_L2.9-W1.6-P0.95-LS2.8-BL, symbol EasyEDA:USBLC6-2SC6
- added IC1: MIE1W0505BGLVH-3R-P, Samacsys:MIE1W0505BGLVH3RP, symbol Samacsys:MIE1W0505BGLVH-3R-P
- added L1, L2: WE-CNSW_1206, Snapeda:WE-CNSW_1206_WE-CNSW_1206, symbol Snapeda:WE-CNSW_1206
- added LED1, LED2: RED, Samacsys:KSEELP4122P1R258A8J8020R18, symbol Samacsys:KS_EELP41.22-P1R2-58-A8J8-020-R18
- added R1, R10, R11, R8, R9: 1K, Samacsys:RESC1608X55N, symbol Samacsys:RT0603FRE071KL
- added R2, R3, R4, R5, R6, R7: 0R, Samacsys:RESC1608X55N, symbol Samacsys:RC0603FR-070RL
- added U1: ADUM3160BRWZ, EasyEDA:WSOIC-16_L10.3-W7.5-P1.27-LS10.3-BL, symbol EasyEDA:ADUM3160BRWZ
- added USB1: USB-B01, EasyEDA:USB-B-TH_USB-B01, symbol EasyEDA:USB-B01
- added USB2: U-USBAR04P-F001, EasyEDA:USB-A-TH_USB-302-T, symbol EasyEDA:U-USBAR04P-F001
Connections:
- new net: R6.1, R7.2, U1.13 (SPD)
- new net: L2.2, R10.1, U1.10 (DD+)
- new net: R8.1, U1.12 (PIN)
- new net: R8.2, U1.14 (VDD2)
- new net: R4.1, R5.2, U1.5 (SPU)
- new net: LED1.2 (A), R1.2
- new net: LED2.2 (A), R11.2
- new net +5V: C1.1 (+), C10.1, C11.1, C2.1, C3.1, D1.5, IC1.10 (VIN_2), IC1.14 (VIN_3), IC1.8 (EN), IC1.9 (VIN_1), R1.1, R4.2, U1.1 (VBUS1), U1.3 (VDD1), U1.4 (PDEN), USB1.1 (VBUS)
- new net D+: D1.3, USB1.3 (D+)
- new net D-: D1.1, USB1.2 (D-)
- new net D1+: D1.4, L1.2, R3.1
- new net D1-: D1.6, L1.3, R2.1
- new net D2+: L1.1, R3.2, U1.7 (UD+)
- new net D2-: L1.4, R2.2, U1.6 (UD-)
- new net D3-: L2.3, R9.1, U1.11 (DD-)
- new net D4+: D2.3, L2.1, R10.2
- new net D4-: D2.1, L2.4, R9.2
- new net D5+: D2.4, USB2.3 (D+)
- new net D5-: D2.6, USB2.2 (D-)
- new net GND: C1.2 (-), C10.2, C11.2, C2.2, C3.2, D1.2, IC1.1 (GND1_1), IC1.11 (GND1_2), IC1.12 (GND1_3), IC1.13 (GND1_4), LED1.1 (K), R5.1, R7.1, U1.2 (GND1), U1.8 (GND1), USB1.4 (GND), USB1.5 (GND), USB1.6 (GND)
- new net GND1: C12.2, C13.2, C14.2 (-), C15.2, C16.2, D2.2, IC1.16 (GND2_4), IC1.2 (GND2_1), IC1.3 (GND2_2), IC1.4 (GND2_3), LED2.1 (K), U1.15 (GND2), U1.9 (GND2), USB2.4 (GND), USB2.5 (SH1), USB2.6 (SH2)
- new net VCC: C12.1, C13.1, C14.1 (+), C15.1, C16.1, D2.5, IC1.15 (VOUT_3), IC1.5 (VOUT_1), IC1.6 (VOUT_2), IC1.7 (VSEL), R11.1, R6.2, U1.16 (VBUS2), USB2.1 (VCC)
Other:
- note added: "DNP"
- company: (none) -> Breiny Feliz / 2023-0545
- title: (none) -> Aislador USB

Commit message: Aislador
Parts:
- removed C1, C14: 470uF/16v, Samacsys:EEE1AA220WR, symbol Samacsys:EEE-FN1C470UR
- removed C10, C11, C12, C13, C15, C3: .1uF, Samacsys:CAPC1608X90N, symbol Samacsys:0603YC104J4T2A
- removed C16, C2: 10uF, Samacsys:CAPC1608X102N, symbol Samacsys:0603YD106KAT2A
- removed D1, D2: USBLC6-2SC6, EasyEDA:SOT-23-6_L2.9-W1.6-P0.95-LS2.8-BL, symbol EasyEDA:USBLC6-2SC6
- removed IC1: MIE1W0505BGLVH-3R-P, Samacsys:MIE1W0505BGLVH3RP, symbol Samacsys:MIE1W0505BGLVH-3R-P
- removed L1, L2: WE-CNSW_1206, Snapeda:WE-CNSW_1206_WE-CNSW_1206, symbol Snapeda:WE-CNSW_1206
- removed LED1, LED2: RED, Samacsys:KSEELP4122P1R258A8J8020R18, symbol Samacsys:KS_EELP41.22-P1R2-58-A8J8-020-R18
- removed R1, R10, R11, R8, R9: 1K, Samacsys:RESC1608X55N, symbol Samacsys:RT0603FRE071KL
- removed R2, R3, R4, R5, R6, R7: 0R, Samacsys:RESC1608X55N, symbol Samacsys:RC0603FR-070RL
- removed U1: ADUM3160BRWZ, EasyEDA:WSOIC-16_L10.3-W7.5-P1.27-LS10.3-BL, symbol EasyEDA:ADUM3160BRWZ
- removed USB1: USB-B01, EasyEDA:USB-B-TH_USB-B01, symbol EasyEDA:USB-B01
- removed USB2: U-USBAR04P-F001, EasyEDA:USB-A-TH_USB-302-T, symbol EasyEDA:U-USBAR04P-F001
- added C10, C11, C4, C5, C6, C7, C8, C9: GRM21BR71H104KA01L, SamacSys_Parts:CAPC2012X145N, symbol SamacSys_Parts:GRM21BR71H104KA01L
- added C2, C3: GRM21BR61C106KE15L, SamacSys_Parts:CAPC2012X145N, symbol SamacSys_Parts:GRM21BR61C106KE15L
- added D1, D2: IR26-21C_L110_TR8, LED_SMD:LED_1206_3216Metric, symbol LED:IR26-21C_L110_TR8
- added IC1: ADUM5000ARWZ, SamacSys_Parts:SOIC127P1032X265-16N, symbol SamacSys_Parts:ADUM5000ARWZ
- added IC2, IC3: NUP2202W1T2G, SamacSys_Parts:SOT65P210X110-6N, symbol SamacSys_Parts:NUP2202W1T2G
- added IC4: ADUM4160BRWZ, SOIC127P1032X265-16N, symbol SamacSys_Parts:ADUM4160BRWZ
- added J1: 87520-0010BLF, SamacSys_Parts:875200010BLF, symbol SamacSys_Parts:87520-0010BLF
- added J2: USB-B-S-F-B-TH-R, SamacSys_Parts:USBBSFBTHR, symbol SamacSys_Parts:USB-B-S-F-B-TH-R
- added R10, R11, R12, R13, R14, R15, R16, R3, R8, R9: ERJ-6GEY0R00V, SamacSys_Parts:RESC2012X70N, symbol SamacSys_Parts:ERJ-6GEY0R00V
- added R2: ERJ-6ENF1002V, SamacSys_Parts:ERJ6ENF1000V, symbol SamacSys_Parts:ERJ-6ENF1002V
Connections:
- net +5V: now also C2.1, C4.1, C5.1, C8.1, C9.1, IC1.8 (GND1_2), IC2.5 (VP), IC4.1 (VBUS1), IC4.3 (VDD1), IC4.4 (PDEN), J1.1, R16.1, R3.1
- net D+: now also IC2.1 (I/O_1), J1.3, R15.1
- net D-: now also IC2.6 (I/O_2), J1.2, R14.1
- net D2+: now also IC4.7 (UD+), R15.2
- net D2-: now also IC4.6 (UD-), R14.2
- net D3-: now also IC4.11 (DD-), R13.1
- net D5+: now also IC3.6 (I/O_2), J2.3, R12.2
- net D5-: now also IC3.1 (I/O_1), J2.2, R13.2
- net GND: now also C2.2, C4.2, C5.2, C8.2, C9.2, D1.1 (K), IC1.1 (VDD1_1), IC1.13 (VSEL), IC2.2 (VN), IC4.2 (GND1_1), IC4.8 (GND1_2), J1.4, J1.MH1, J1.MH2, R10.2, R8.2
- net GND1: now also C10.2, C11.2, C3.2, C6.2, C7.2, D2.1 (K), IC1.2 (GND1_1), IC1.9 (GNDISO_1), IC3.2 (VN), IC4.15 (GND2_2), IC4.9 (GND2_1), J2.4, J2.MH1, J2.MH2
- net VCC: now also C10.1, C11.1, C3.1, C6.1, C7.1, IC1.10 (VISO_1), IC1.11 (NC_2), IC1.15 (GNDISO_2), IC1.16 (VISO_2), IC1.6 (RCSEL), IC1.7 (VDD1_2), IC3.5 (VP), IC4.16 (VBUS2), J2.1, R11.1, R9.1
- new net: D2.2 (A), R11.2
- new net: D1.2 (A), R16.2
- new net: IC4.5 (SPU), R3.2, R8.1
- new net: IC4.13 (SPD), R10.1, R9.2
- new net: IC4.10 (DD+), R12.1
- new net: IC4.12 (PIN), R2.2
- new net: IC4.14 (VDD2), R2.1
- no-connect marks 0 -> 9
